File: CAN-Sensor-Hub-v1.kicad_sch (KiCad schematic)
At the start: 57 parts, among them J1 Conn_01x04, J2 Conn_01x04, J3 Conn_01x04, J4 USB_C_Receptacle_USB2.0_14P, J5 Conn_ARM_JTAG_SWD_10, J6 Conn_01x04, J7 Conn_01x04, SW1 NRST, SW2 BOOT, U1 TPS5430DDA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

Commit message: Cleaned up schematic, added 5V->3V linear converter
Parts:
- removed C8: 10nF, symbol Device:C_Small
- removed C9: 100uF, symbol Device:C_Small_US
- removed D7: D_Schottky, symbol Device:D_Schottky
- removed JP1, JP2, JP3, JP4: ~, symbol Jumper:Jumper_2_Small_Open
- removed L2: 15uH, symbol Device:L
- removed R12: 10k, symbol Device:R_Small_US
- removed R13: 5.9k, symbol Device:R_Small_US
- removed R4, R5, R6, R7: 4.7k, symbol Device:R_US
- removed U4: TPS5430DDA, Package_SO:TI_SO-PowerPAD-8_ThermalVias, symbol Regulator_Switching:TPS5430DDA
- added C17, C18: 10uF, symbol Device:C_Small
- added C19: 100nF, symbol Device:C_Small
- added U4: AZ1117-3.3, symbol Regulator_Linear:AZ1117-3.3
Connections:
- net GNDREF: now also D1.1 (K), D2.1 (K), D3.1 (K), C17.2, C18.2, C19.2, U4.1 (GND)
- net I2C1_SCL: now also J1.4 (Pin_4)
- net I2C1_SDA: now also J1.3 (Pin_3)
- net I2C2_SCL: no longer J1.4 (Pin_4)
- net I2C2_SDA: no longer J1.3 (Pin_3)
- net VDD_3V3: now also C17.1, C19.1, U4.2 (VO)
- net VDD_5V: now also C18.1, U4.3 (VI)
- net VIN_12V renamed VBAT_12V
Other:
- note added: "12V ---------------------> 5V"
- note added: "12V->5V DC/DC Buck Converter"
- note added: "3.3V/1A"
- note added: "32.768KHz Crystal"
- note added: "5.1k pulldown resistors on CC pins to identify as device mode Should we have some way to switch to host mode? We could have a transistor controlled by a GPIO pin that can change these resistors from pullup to pulldown Or we could use a dual-role IC but that's expensive.."
- note added: "5V --------------------> 3.3V"
- note added: "5V->3.3V DC/DC Linear Converter"
- note added: "5V/3A"
- note added: "8MHz Crystal"
- note added: "CAN BUS TRANSCEIVER AND CONNECTORS"
- note added: "CODE BLUE"
- note added: "Crystal cap values taken from STM32F722 Nucleo board schematic"
- note added: "Decoupling capacitors"
- note added: "Design is based on example 12V-5V/3A converter circuit in TPS5430DDA datasheet. https://www.ti.com/lit/ds/symlink/tps5430.pdf?ts=1750604171587&ref_url=https%253A%252F%252Fwww.google.com%252F Section 7.2 - Typical Applications"
- note added: "Design taken from example in AZ1117-3.3 datasheet"
- note added: "JTAG/SWD Debug Port"
- note added: "Microcontroller"
- note added: "One 100nF cap per VDD pin to handle high frequency noise One 4.7uF bulk cap for voltage dips"
- note added: "POWER SUPPLY"
- note added: "PWR RED"
- note added: "QSPI FLash Extra storage for code / libraries / logs"
- note added: "Status LEDs"
- note added: "TODO: Calculate series resistor values that will allow us to drive these LEDs from a GPIO pin on the STM32F722."
- note added: "TODO: Isolate VDDA from VDD through a ferrite bead (saw this in STM32 power docs..)"
- note added: "TODO: Need to take connector layout from CDB design"
- note added: "USB-C Connector"
- note added: "USER GREEN"
- note removed: "TODO: Figure out what to do with WPn and RESETn lines"
- moved on the sheet: C1, C10, C11, C12, C13, C14, C15, C16, C2, C3, C4, C5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

Commit message: Updated schematic, added PCB file with footprints assigned and started experimenting
Parts:
- added J10, J11, J9: Conn_01x03, Connector_PinHeader_2.54mm:PinHeader_1x03_P2.54mm_Horizontal, symbol Connector_Generic:Conn_01x03
- added J8: Conn_01x04, TerminalBlock_WAGO:TerminalBlock_WAGO_2601-1104_1x04_P3.50mm_Horizontal, symbol Connector_Generic:Conn_01x04
- added Q1, Q2: NMOS, Package_TO_SOT_SMD:SOT-23, symbol Simulation_SPICE:NMOS
- added R12, R13, R14, R15, R16: 10k, Resistor_SMD:R_0402_1005Metric, symbol Device:R_Small_US
- C1, C10, C11, C12, C13, C14, C15, C16, C17, C18, C19, C2, C3, C4, C5, C6, C7: footprint (none) -> Capacitor_SMD:C_0402_1005Metric
- D1, D2, D3: footprint (none) -> LED_SMD:LED_0201_0603Metric
- D5, D6: footprint (none) -> Diode_SMD:D_0603_1608Metric
- J1, J2, J3: footprint (none) -> Connector_JST:JST_SH_SM04B-SRSS-TB_1x04-1MP_P1.00mm_Horizontal
- J4: footprint (none) -> Connector_USB:USB_C_Receptacle_GCT_USB4110
- J5: footprint (none) -> Connector_PinHeader_1.27mm:PinHeader_2x05_P1.27mm_Vertical_SMD
- J6, J7: footprint (none) -> TerminalBlock_WAGO:TerminalBlock_WAGO_2601-1104_1x04_P3.50mm_Horizontal
- L1: footprint (none) -> Inductor_SMD:L_0402_1005Metric
- R1, R10, R11, R2, R3, R8, R9: footprint (none) -> Resistor_SMD:R_0402_1005Metric
- SW1, SW2: footprint (none) -> lib:SW_TS-1088-AR02016
- U2: footprint (none) -> Package_SO:SOIC-8_3.9x4.9mm_P1.27mm
- U4: footprint (none) -> Package_TO_SOT_SMD:SOT-223-3_TabPin2
- X1: footprint (none) -> Crystal:Crystal_SMD_3225-2Pin_3.2x2.5mm
- X2: footprint (none) -> Crystal:Crystal_SMD_3215-2Pin_3.2x1.5mm
Connections:
- net CAN1_RX is gone; now on net CAN_RX: U7.70 (PA11)
- net CAN1_TX is gone; now on net CAN_TX: U7.71 (PA12)
- net GNDREF: now also J7.4 (Pin_4), U2.8 (STB), J10.3 (Pin_3), J11.3 (Pin_3), J8.4 (Pin_4), J9.3 (Pin_3); no longer C17.2, C18.2, U4.1 (GND)
- net QSPI_NCS: now also R16.2
- net USART2_RX: now also J11.2 (Pin_2)
- net USART2_TX: now also J11.1 (Pin_1)
- net VBAT_12V: now also J7.3 (Pin_3), J8.3 (Pin_3)
- net VDD_3V3: now also U2.5 (VIO), Q1.2 (G), Q2.2 (G), R12.1, R14.1, R16.1
- net VDD_5V: now also J10.2 (Pin_2), J9.2 (Pin_2), R13.1, R15.1
- net DIO_0_3V3: now reaches U7.81 (PD0)
- net DIO_0_3V3: now also Q1.3 (S), R12.2
- net DIO_1_3V3: now reaches U7.82 (PD1)
- net DIO_1_3V3: now also Q2.3 (S), R14.2
- net CAN_H: now reaches J6.1 (Pin_1)
- net CAN_H: now also J6.3 (Pin_3), J7.1 (Pin_1), U2.7 (CANH), J8.1 (Pin_1)
- net CAN_L: now reaches J6.2 (Pin_2)
- net CAN_L: now also J6.4 (Pin_4), J7.2 (Pin_2), U2.6 (CANL), J8.2 (Pin_2)
- new net: C17.2, C18.2, U4.1 (GND)
- new net DIO_0_5V: J10.1 (Pin_1), Q1.1 (D), R13.2
- new net DIO_1_5V: J9.1 (Pin_1), Q2.1 (D), R15.2
Other:
- note added: "3V3 to 5V level shifters"
- note added: "DIO Ports"
- note added: "Downstream / Motor CAN"
- note added: "JTAG/SWD and UART Debug Port"
- note added: "Male 3-pin 2.54mm headers (same as RoboRIO)"
- note added: "Motor CAN"
- note added: "Power IN"
- note added: "Power OUT"
- note added: "SWD Debug Port"
- note added: "UART Debug"
- note added: "Upstream CAN"
- note added: "YEL GRN RED BLK"
- note added: "YEL GRN YEL GRN"
- note added: "https://www.st.com/resource/en/application_note/an4760-quadspi-interface-on-stm32-microcontrollers-and-microprocessors--stmicroelectronics.pdf"
- note removed: "JTAG/SWD Debug Port"
- moved on the sheet: J6, J7, U3

Commit message: Initial prototype layout done - likely needs to be redone
Parts:
- added C20: 4.7uF, Capacitor_SMD:C_0603_1608Metric, symbol Device:C_Small
- added C21: 100nF, Capacitor_SMD:C_0402_1005Metric, symbol Device:C_Small
- added C23, C24: 10uF, Capacitor_SMD:C_0603_1608Metric, symbol Device:C_Small
- added Q3: PMOS, Package_TO_SOT_SMD:SOT-23, symbol Simulation_SPICE:PMOS
- C15, C17, C18: footprint Capacitor_SMD:C_0402_1005Metric -> Capacitor_SMD:C_0603_1608Metric
- C16, C7: footprint Capacitor_SMD:C_0402_1005Metric -> Capacitor_SMD:C_0805_2012Metric
- D1, D2, D3: footprint LED_SMD:LED_0201_0603Metric -> LED_SMD:LED_0805_2012Metric
- J11: footprint Connector_PinHeader_2.54mm:PinHeader_1x03_P2.54mm_Horizontal -> Connector_PinHeader_2.54mm:PinHeader_1x03_P2.54mm_Vertical
- L1: footprint Inductor_SMD:L_0402_1005Metric -> Inductor_SMD:L_Sumida_CDMC6D28_7.25x6.5mm
Connections:
- net CAN_H: now also J8.3 (Pin_3); no longer J8.1 (Pin_1)
- net CAN_L: now also J8.4 (Pin_4); no longer J8.2 (Pin_2)
- net GNDREF: now also C17.2, C18.2, J8.2 (Pin_2), U4.1 (GND), C20.2, C21.2, C23.2, C24.2; no longer J8.4 (Pin_4)
- net VBAT_12V: now also J8.1 (Pin_1); no longer J8.3 (Pin_3)
- net VBUS_5V: now also C20.1, Q3.2 (G)
- net VDD_5V: now also C21.1, C23.1, C24.1, Q3.3 (S); no longer C7.1, L1.2, R8.1
- new net: C7.1, L1.2, Q3.1 (D), R8.1
Other:
- note added: "CODE WHITE"
- note added: "From RPi doc: An example of a suitable P-MOSFET for most situations is Diodes DMG2305UX which has a maximum Vt of 0.9V and Ron of 100mΩ (at 2.5V Vgs)."
- note added: "RED BLK YEL GRN"
- note added: "TODO: What are these VCAP pins? They weren't present on the LQFP64 version of the part"
- note added: "TODO: What is VREF+?"
- note added: "This PMOS transistor turns off the 12->5V supply when 5V is applied to the USB port. This ensures that we don't pump current *into* your laptop's USB port."
- note added: "This part # should be TCAN1042VDRQ1 The "V" Suffix provides level shifting through VIO pin"
- note added: "USB PWR IN ->"
- note removed: "CODE BLUE"
- note removed: "TODO: Need to take connector layout from CDB design"
- moved on the sheet: D5, J1, J2, J3, J6, J7, J8

Commit message: V0.2 of board, nearly ready for production
Parts:
- removed J6, J7, J8: Conn_01x04, TerminalBlock_WAGO:TerminalBlock_WAGO_2601-1104_1x04_P3.50mm_Horizontal, symbol Connector_Generic:Conn_01x04
- removed SW2: BOOT, lib:SW_TS-1088-AR02016, symbol Switch:SW_Push
- added C22, C25, C26: 100nF, Capacitor_SMD:C_0402_1005Metric, symbol Device:C_Small
- added C8, C9: 2.2uF, Capacitor_SMD:C_0402_1005Metric, symbol Device:C_Small
- added H1, H2, H3, H4: MountingHole, MountingHole:MountingHole_2.7mm_M2.5, symbol Mechanical:MountingHole
- added J12: Conn_01x12, TerminalBlock_WAGO:TerminalBlock_WAGO_2601-1112_1x12_P3.50mm_Horizontal, symbol Connector_Generic:Conn_01x12
- added J6: Conn_01x02, Connector_PinHeader_2.54mm:PinHeader_1x02_P2.54mm_Vertical, symbol Connector_Generic:Conn_01x02
- added R4, R6: 160, Resistor_SMD:R_0402_1005Metric, symbol Device:R_Small_US
- added R5: 60, Resistor_SMD:R_0402_1005Metric, symbol Device:R_Small_US
Connections:
- net CAN_H: now also J12.3 (Pin_3), J12.5 (Pin_5), J12.7 (Pin_7), J12.9 (Pin_9)
- net CAN_L: now also J12.10 (Pin_10), J12.4 (Pin_4), J12.6 (Pin_6), J12.8 (Pin_8)
- net GNDREF: now also C22.2, C25.2, C26.2, C8.2, C9.2, J12.12 (Pin_12), J12.2 (Pin_2), J6.1 (Pin_1)
- net USART2_RX: now also J11.1 (Pin_1); no longer J11.2 (Pin_2)
- net USART2_TX: now also J11.2 (Pin_2); no longer J11.1 (Pin_1)
- net VBAT_12V: now also J12.1 (Pin_1), J12.11 (Pin_11)
- net VDD_3V3: now also C22.1, C25.1, C26.1, R4.1
- net at D3.2 (A): now also R5.2
- net IO_LED3: now reaches U7.37 (PE7)
- net IO_LED3: now also R6.1
- net IO_LED2: now reaches U7.38 (PE8)
- net IO_LED2: now also R5.1
- net IO_LED1: now reaches U7.39 (PE9)
- net at U7.48 (VCAP_1): now also C9.1
- net at U7.73 (VCAP_2): now also C8.1
- net at U7.94 (BOOT0): now also J6.2 (Pin_2)
- net at D1.2 (A): now also R6.2
- net at D2.2 (A): now also R4.2
Other:
- note removed: "TODO: What are these VCAP pins? They weren't present on the LQFP64 version of the part"
- note removed: "TODO: What is VREF+?"
- moved on the sheet: D1, D2, D3

Commit message: Production ready board
Parts:
- added C27: 100nF, Capacitor_SMD:C_0402_1005Metric, symbol Device:C_Small
- added R17: 10k, Resistor_SMD:R_0402_1005Metric, symbol Device:R_Small_US
- added R18: 100k, Resistor_SMD:R_0402_1005Metric, symbol Device:R_Small_US
- added TP1, TP10, TP11, TP12, TP13, TP14, TP15, TP16, TP17, TP18, TP19, TP2, TP20, TP3, TP4, TP5, TP6, TP7, TP8, TP9: TestPoint_Small, TestPoint:TestPoint_Pad_D0.5mm, symbol Connector:TestPoint_Small
- C1, C2: value 10pF -> 4.3pF; LCSC (none) -> CL05C100JB5NNNC
- C10, C11, C12, C13, C14, C19, C21, C22, C25, C26, C5: LCSC (none) -> CL05B104KO5NNNC
- C15, C20: LCSC (none) -> CL10A475KO8NNNC
- C16: LCSC (none) -> CL21A475KAQNNNE
- C17, C18, C23, C24: LCSC (none) -> CL10A106MA8NRNC
- C3, C4: LCSC (none) -> 0402CG2R0C500NT
- C6: LCSC (none) -> CL05B103KB5NNNC
- C7: footprint Capacitor_SMD:C_0805_2012Metric -> Capacitor_Tantalum_SMD:CP_EIA-3528-21_Kemet-B
- C8, C9: LCSC (none) -> CL05A225MQ5NSNC
- D1: LCSC (none) -> KT-0805G
- D2: LCSC (none) -> NCD0805R1
- D3: LCSC (none) -> KT-0805W
- D5, D6: LCSC (none) -> SD0603S040S0R2
- J1, J2, J3: LCSC (none) -> SM04B-SRSS-TB(LF)(SN)
- J10, J11, J12, J5, J9: now not fitted; now left out of the parts list
- J4: LCSC (none) -> TYPEC-304YSSW-ACP16
- L1: LCSC (none) -> CYA0650-15UH
- Q1, Q2: LCSC (none) -> SI2301CDS-T1-GE3
- Q3: LCSC (none) -> AO3401A
- R1, R2, R3: footprint Resistor_SMD:R_0402_1005Metric -> Resistor_SMD:R_0805_2012Metric; now not fitted; now left out of the parts list
- R10, R9: LCSC (none) -> 0402WGF5101TCE
- R11: LCSC (none) -> 0402WGF3241TCE
- R12, R13, R14, R15, R8: LCSC (none) -> 0402WGF1002TCE
- R4: value 160 -> 100; LCSC (none) -> 0402WGF1000TCE
- R5: value 60 -> 100; LCSC (none) -> 0402WGF1000TCE
- R6: value 160 -> 150; LCSC (none) -> 0402WGF1500TCE
- SW1: LCSC (none) -> TS-1088-AR02016
- U1: LCSC (none) -> TPS5430DDAR
- U2: LCSC (none) -> https://jlcpcb.com/partdetail/TexasInstruments-TCAN1042VDRQ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
- U3: LCSC (none) -> W25Q32JVZPIQ
- U4: LCSC (none) -> AMS1117-3.3
- U7: LCSC (none) -> STM32F722VET6
- X1: LCSC (none) -> NX3225GD-8MHZ-STD-CRA-3
- X2: LCSC (none) -> NX3215SA-32.768K-STD-MUA-14
Connections:
- net CAN_RX: now also TP11.1
- net CAN_TX: now also TP12.1
- net GNDREF: now also C27.2, R17.1; no longer J6.1 (Pin_1)
- net I2C1_SCL: now also TP14.1
- net I2C1_SDA: now also TP13.1
- net I2C2_SCL: now also TP16.1
- net I2C2_SDA: now also TP15.1
- net I2C3_SCL: now also TP18.1
- net I2C3_SDA: now also TP17.1
- net OTG_HS_DM: now also TP7.1
- net OTG_HS_DP: now also TP8.1
- net QSPI_CLK: now also TP2.1
- net QSPI_IO0: now also TP3.1
- net QSPI_IO1: now also TP4.1
- net QSPI_IO2: now also TP5.1
- net QSPI_IO3: now also TP6.1
- net QSPI_NCS: now also TP1.1
- net USART2_RX: now also TP19.1
- net USART2_TX: now also TP20.1
- net VDD_3V3: now also C27.1, R18.2, TP10.1
- net VDD_5V: now also TP9.1
- net at J6.2 (Pin_2), U7.94 (BOOT0): now also R18.1
- new net: J6.1 (Pin_1), R17.2
Other:
- moved on the sheet: J6
